File: ecad/ecad.kicad_sch (KiCad schematic)
At the start: 22 parts, among them J1 Raspberry_Pi_2_3, Q1 BC547, Q4 BC547, SW1 Power Button, U2 USB PD/QC Decoy, U3 VRB1205YMD_6wr3, U6 Power Bank

Commit message: Add volume buttons and led to schematic (#35)
* Added volume buttons.

* Added status LED circuit.

* Some annotations.

* Changed LED library element.

* Replaced wrong +5V supply elements with +5VD

* Updated schematics
Parts:
- added D1: LED, symbol Device:LED
- added Q2: BC547, Package_TO_SOT_THT:TO-92_Inline, symbol Transistor_BJT:BC547
- added R7: 100, symbol Device:R
- added R8: 30k, symbol Device:R
- added SW2, SW3: SW_Push, symbol Switch:SW_Push
Connections:
- net +5V is gone; now on net +5VD: C2.1, U3.3 (+Vo)
- net +5VD: now also R7.2
- net GNDD: now also Q2.3 (E), SW2.2, SW3.2
- net VOLUME_DOWN: now reaches J1.11 (GPIO17)
- net VOLUME_DOWN: now also SW2.1
- net VOLUME_UP: now reaches J1.13 (GPIO27)
- net VOLUME_UP: now also SW3.1
- net STATUS_LED: now reaches J1.32 (PWM0/GPIO12)
- net STATUS_LED: now also R8.2
- new net: Q2.2 (B), R8.1
- new net: D1.1 (K), Q2.1 (C)
- new net: D1.2 (A), R7.1
Other:
- note added: "Assuming white LED with 4V/10mA flux voltage and current"
- note added: "Status LED Should at some point indicate operational state (e.g., booting up, shutting down, bluetooth pairing, no internet,...)"
- moved on the sheet: Q1, Q4, R1, R2
